Commit message: 251204

File: urdf/common/camera.urdf.xacro (robot description, xacro)
@@ -11,5 +11,6 @@
                 <origin xyz="0 0 0" rpy="0 0 0"/>
                 <geometry>
-                    <mesh filename="package://rm_description/meshes/common/camera.stl" scale="0.001 0.001 0.001"/>
+                    <mesh filename="package://rm_description/meshes/common/camera.stl"
+                    		scale="0.001 0.001 0.001"/>
                 </geometry>
             </visual>
